Commit message: Real Sense Added, Image not Publishing

File: bat_algo/urdf/small_bot.xacro (robot description, xacro)
@@ -1,4 +1,5 @@
 <?xml version="1.0"?>
 <robot xmlns:xacro="http://www.ros.org/wiki/xacro" name="$(arg robot_name)">
+<xacro:include filename="$(find realsense2_description)/urdf/_d435.urdf.xacro"/>
     <link name="base_link">
         <visual>
@@ -117,4 +118,7 @@
         </inertial>
     </link>
+    <xacro:sensor_d435 name="camera" topics_ns="camera" parent="base_link" publish_pointcloud="true">
+        <origin xyz="0 0 0.05" rpy="0 0 0" />
+    </xacro:sensor_d435>
     <joint name="front_wheel_joint" type="fixed">  <!-- continuous -->
         <axis xyz="0.0 0.0 1"/>

Commit message: Revert "Real Sense Added, Image not Publishing"
This reverts commit 7a3d5c1d88364c5f763735d5046f0b0c891688fe.

File: bat_algo/urdf/small_bot.xacro (robot description, xacro)
@@ -1,5 +1,4 @@
 <?xml version="1.0"?>
 <robot xmlns:xacro="http://www.ros.org/wiki/xacro" name="$(arg robot_name)">
-<xacro:include filename="$(find realsense2_description)/urdf/_d435.urdf.xacro"/>
     <link name="base_link">
         <visual>
@@ -118,7 +117,4 @@
         </inertial>
     </link>
-    <xacro:sensor_d435 name="camera" topics_ns="camera" parent="base_link" publish_pointcloud="true">
-        <origin xyz="0 0 0.05" rpy="0 0 0" />
-    </xacro:sensor_d435>
     <joint name="front_wheel_joint" type="fixed">  <!-- continuous -->
         <axis xyz="0.0 0.0 1"/>

Commit message: Camera Image Publishing, teleop twist has issues

File: bat_algo/urdf/small_bot.xacro (robot description, xacro)
@@ -2,4 +2,5 @@
 <robot xmlns:xacro="http://www.ros.org/wiki/xacro" name="$(arg robot_name)">
 <xacro:include filename="$(find realsense2_description)/urdf/_d435.urdf.xacro"/>
+<xacro:property name="cam_topic" value="$(arg robot_name)" />
     <link name="base_link">
         <visual>
@@ -118,5 +119,5 @@
         </inertial>
     </link>
-    <xacro:sensor_d435 name="camera" topics_ns="camera" parent="base_link" publish_pointcloud="true">
+    <xacro:sensor_d435 name="camera" topics_ns="${cam_topic}/camera" parent="base_link" publish_pointcloud="true">
         <origin xyz="0 0 0.05" rpy="0 0 0" />
     </xacro:sensor_d435>
